Commit message: rename third_robot to cirkit_unit03

File: cirkit_unit03_description/urdf/cirkit_unit03.urdf (robot description, URDF)
Before this commit: robot origins, 9 links, 8 joints
Links:
- link base_link: geometry visual mesh filename=package://cirkit_unit03_description/meshes/cirkit_unit03/ci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
- link front_bottom_lrf: geometry visual mesh filename=package://cirkit_unit03_description/meshes/LRF/UTM-30LX.dae
- link front_top_3durg: geometry visual mesh filename=package://cirkit_unit03_description/meshes/3DURG/hokuyo3dur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
- link left_front_wheel: geometry visual mesh filename=package://cirkit_unit03_description/meshes/cirkit_unit03/ci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
- link left_rear_wheel: geometry visual mesh filename=package://cirkit_unit03_description/meshes/cirkit_unit03/ci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
- link rear_bottom_lrf: geometry visual mesh filename=package://cirkit_unit03_description/meshes/LRF/UTM-30LX.dae
- link right_front_wheel: geometry visual mesh filename=package://cirkit_unit03_description/meshes/cirkit_unit03/ci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
- link right_rear_wheel: geometry visual mesh filename=package://cirkit_unit03_description/meshes/cirkit_unit03/ci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

File: cirkit_unit03_description/urdf/cirkit_unit03.xacro (robot description, xacro)
@@ -3,14 +3,14 @@
     <xacro:property name="camera_link" value="0.05" /> <!-- Size of square 'camera' box -->
     <!-- Import all Gazebo-customization elements, including Gazebo colors -->
-    <xacro:include filename="$(find third_robot_description)/urdf/third_robot.gazebo" />
+    <xacro:include filename="$(find cirkit_unit03_description)/urdf/cirkit_unit03.gazebo" />
     <!-- Import Rviz colors -->
-    <xacro:include filename="$(find third_robot_description)/urdf/materials.xacro" />
+    <xacro:include filename="$(find cirkit_unit03_description)/urdf/materials.xacro" />
     <!-- Import macros -->
-    <xacro:include filename="$(find third_robot_description)/urdf/third_robot_macro.xacro" />
+    <xacro:include filename="$(find cirkit_unit03_description)/urdf/cirkit_unit03_macro.xacro" />
     <link name="base_link">
       <visual>
         <origin rpy="0 0 0" xyz="0 0 0.55" />
         <geometry>
-          <mesh filename="package://third_robot_description/meshes/third_robot/third_robot_body.dae"/>
+          <mesh filename="package://cirkit_unit03_description/meshes/cirkit_unit03/cirkit_unit03_body.dae"/>
         </geometry>
       </visual>
@@ -33,5 +33,5 @@
     <!--         <origin rpy="0 0.5 0" xyz="0 0 0"/> -->
     <!--         <geometry> -->
-    <!--             <mesh filename="package://third_robot_description/meshes/LRF/UTM-30LX.dae"/> -->
+    <!--             <mesh filename="package://cirkit_unit03_description/meshes/LRF/UTM-30LX.dae"/> -->
     <!--         </geometry> -->
     <!--     </visual> -->
@@ -48,5 +48,5 @@
         <origin rpy="0 0 0" xyz="-0.10 0 0"/>
         <geometry>
-          <mesh filename="package://third_robot_description/meshes/3DURG/hokuyo3durg.dae"/>
+          <mesh filename="package://cirkit_unit03_description/meshes/3DURG/hokuyo3durg.dae"/>
         </geometry>
       </visual>
@@ -70,5 +70,5 @@
         <origin rpy="0 0 0" xyz="0 0 0"/>
         <geometry>
-          <mesh filename="package://third_robot_description/meshes/LRF/UTM-30LX.dae"/>
+          <mesh filename="package://cirkit_unit03_description/meshes/LRF/UTM-30LX.dae"/>
         </geometry>
       </visual>
@@ -94,5 +94,5 @@
             <origin rpy="0 0 0" xyz="0 0 0"/>
             <geometry>
-                <mesh filename="package://third_robot_description/meshes/LRF/UTM-30LX.dae"/>
+                <mesh filename="package://cirkit_unit03_description/meshes/LRF/UTM-30LX.dae"/>
             </geometry>
         </visual>
@@ -116,5 +116,5 @@
         <origin rpy="0 0 ${PI}" xyz="0 0 0"/>
         <geometry>
-          <mesh filename="package://third_robot_description/meshes/LRF/UTM-30LX.dae"/>
+          <mesh filename="package://cirkit_unit03_description/meshes/LRF/UTM-30LX.dae"/>
         </geometry>
       </visual>

File: cirkit_unit03_description/urdf/cirkit_unit03_macro.xacro (robot description, xacro)
@@ -27,5 +27,5 @@
                 <!-- <origin rpy="${PI/2-reflect_right_left*PI/2} 0 0" xyz="0 0 0"/> -->
                 <geometry>
-                    <mesh filename="package://third_robot_description/meshes/third_robot/third_robot_wheel.dae"/>
+                    <mesh filename="package://cirkit_unit03_description/meshes/cirkit_unit03/cirkit_unit03_wheel.dae"/>
                 </geometry>
                 ->
@@ -79,5 +79,5 @@
                 <!-- <origin rpy="${PI/2-reflect_right_left*PI/2} 0 0" xyz="0 0 0"/> -->
                 <geometry>
-                    <mesh filename="package://third_robot_description/meshes/third_robot/third_robot_wheel.dae"/>
+                    <mesh filename="package://cirkit_unit03_description/meshes/cirkit_unit03/cirkit_unit03_wheel.dae"/>
                 </geometry>
                 ->
