Commit message: Update xacro model for new steer_drive configuration.

File: cirkit_unit03_description/urdf/cirkit_unit03.xacro (robot description, xacro)
@@ -23,5 +23,5 @@
       <xacro:default_inertial mass="10"/>
     </link>
-    <!-- wheels -->
+    <xacro:rear_wheel/>
     <xacro:front_wheel right_left="right" reflect_right_left="1"/>
     <xacro:front_wheel right_left="left" reflect_right_left="-1"/>
@@ -81,9 +81,9 @@
     </joint>
     <!-- steer -->
-    <link name="steer"/>
-    <joint name="base_to_steer" type="fixed">
+    <link name="front_steer_link"/>
+    <joint name="front_steer_joint" type="fixed">
         <axis xyz="0 1 0"/>
         <parent link="base_link"/>
-        <child link="steer"/>
+        <child link="front_steer_link"/>
         <origin xyz="0.41 0 0.14"/>
     </joint>

File: cirkit_unit03_description/urdf/cirkit_unit03_macro.xacro (robot description, xacro)
@@ -20,4 +20,14 @@
     </xacro:macro>
     <!-- wheel macro -->
+    <xacro:macro name="rear_wheel">
+        <link name="rear_wheel_link"/>
+        <joint name="rear_wheel_joint" type="continuous">
+            <axis xyz="0 1 0"/>
+            <parent link="base_link"/>
+            <child link="rear_wheel_link"/>
+            <origin xyz="${-base_center_x-length_from_base_center_to_wheel_x} 0 ${radius_wheel}"/>
+            <origin xyz="${length_from_base_to_wheel_front_x} 0 ${radius_wheel}"/>
+        </joint>
+    </xacro:macro>
     <xacro:macro name="wheel" params="right_left reflect_right_left front_rear reflect_front_rear">
         <link name="${right_left}_${front_rear}_wheel">
@@ -29,5 +39,4 @@
                     <mesh filename="package://cirkit_unit03_description/meshes/cirkit_unit03/cirkit_unit03_wheel.dae"/>
                 </geometry>
-                ->
             </visual>
             <collision>
@@ -67,9 +76,11 @@
             </inertial>
         </link>
-        <joint name="base_to_${right_left}_front_steer" type="continuous">
+        <joint name="base_to_${right_left}_front_steer" type="revolute">
             <axis xyz="0 0 1"/>
             <parent link="base_link"/>
             <child link="steer_${right_left}"/>
-        <origin xyz="${base_center_x+length_from_base_center_to_wheel_x} ${-reflect_right_left*length_from_base_to_wheel_y} 0.30"/>
+            <origin xyz="${base_center_x+length_from_base_center_to_wheel_x} ${-reflect_right_left*length_from_base_to_wheel_y} 0.30"/>
+            <dynamics damping="0.7" friction="0.7"/>
+            <limit effort="7.0" lower="${-80*PI/180}" upper="${80*PI/180}" velocity="${200.0*PI/180.0*0.95}"/>
         </joint>
         <link name="${right_left}_front_wheel">
@@ -81,5 +92,4 @@
                     <mesh filename="package://cirkit_unit03_description/meshes/cirkit_unit03/cirkit_unit03_wheel.dae"/>
                 </geometry>
-                ->
             </visual>
             <collision>

Commit message: Fix xacro config for kinetic

File: cirkit_unit03_description/urdf/cirkit_unit03.xacro (robot description, xacro)
@@ -159,23 +159,3 @@
     <link name="merged_lrf">
     </link>
-    <transmission name="tran1">
-      <type>transmission_interface/SimpleTransmission</type>
-        <joint name="base_to_left_rear_wheel">
-          <hardwareInterface>EffortJointInterface</hardwareInterface>
-        </joint>
-        <actuator name="motor1">
-          <hardwareInterface>EffortJointInterface</hardwareInterface>
-          <mechanicalReduction>1</mechanicalReduction>
-        </actuator>
-    </transmission>
-    <transmission name="tran2">
-      <type>transmission_interface/SimpleTransmission</type>
-      <joint name="base_to_right_rear_wheel">
-        <hardwareInterface>EffortJointInterface</hardwareInterface>
-      </joint>
-      <actuator name="motor2">
-        <hardwareInterface>EffortJointInterface</hardwareInterface>
-        <mechanicalReduction>1</mechanicalReduction>
-      </actuator>
-    </transmission>
 </robot>

File: cirkit_unit03_description/urdf/cirkit_unit03_macro.xacro (robot description, xacro)
@@ -8,5 +8,5 @@
     <xacro:property name="base_center_x" value="0.015" />
     <xacro:property name="length_from_base_center_to_wheel_x" value="0.395" />
-    <xacro:property name="length_from_base_to_wheel_front_x" value="0.41" />
+    <xacro:property name="length_from_base_to_wheel_front_x" value="0.43" />
     <xacro:property name="length_from_base_to_wheel_rear_x" value="0.38" />
     <xacro:property name="length_from_base_to_wheel_y" value="0.25" />
@@ -105,5 +105,10 @@
                 </geometry>
             </collision>
-            <xacro:default_inertial mass="1"/>
+            <inertial>
+                <mass value="0.5" />
+                <inertia ixx="0.02" ixy="0.0" ixz="0.0"
+                    iyy="0.02" iyz="0.0"
+                    izz="0.02" />
+            </inertial>
         </link>
         <joint name="base_to_${right_left}_front_wheel" type="continuous">
