Commit message: Fix xacro for default steer_drive configuration.

File: cirkit_unit03_description/urdf/cirkit_unit03_macro.xacro (robot description, xacro)
@@ -21,5 +21,12 @@
     <!-- wheel macro -->
     <xacro:macro name="rear_wheel">
-        <link name="rear_wheel_link"/>
+        <link name="rear_wheel_link">
+            <collision>
+                <origin rpy="${PI/2} 0 0" xyz="0 0 0"/>
+                <geometry>
+                    <cylinder length="${length_wheel}" radius="${radius_wheel}"/>
+                </geometry>
+            </collision>
+        </link>
         <joint name="rear_wheel_joint" type="continuous">
             <axis xyz="0 1 0"/>
@@ -27,5 +34,4 @@
             <child link="rear_wheel_link"/>
             <origin xyz="${-base_center_x-length_from_base_center_to_wheel_x} 0 ${radius_wheel}"/>
-            <origin xyz="${length_from_base_to_wheel_front_x} 0 ${radius_wheel}"/>
         </joint>
     </xacro:macro>

Commit message: Modify front wheel inertia for kinetic gazebo

File: cirkit_unit03_description/urdf/cirkit_unit03_macro.xacro (robot description, xacro)
@@ -107,7 +107,7 @@
             <inertial>
                 <mass value="0.5" />
-                <inertia ixx="0.02" ixy="0.0" ixz="0.0"
-                    iyy="0.02" iyz="0.0"
-                    izz="0.02" />
+                <inertia ixx="0.50" ixy="0.0" ixz="0.0"
+                    iyy="0.50" iyz="0.0"
+                    izz="0.50" />
             </inertial>
         </link>
